Commit message: add bounding boxes to the feet. Drastically increase the simulation speed. Bullet collision is a lot slower...

File: data/urdf/BioloidGP/BioloidGP.URDF (robot description, URDF)
Before this commit: robot BioloidGP, 17 links, 16 joints
Links:
- link l_foot: geometry collision mesh filename=l_foot_box.obj; visual mesh filename=l_foot.STL
- link r_foot: geometry collision mesh filename=r_foot_box.obj; visual mesh filename=r_foot.STL

Commit message: remove the battery from the urdf files.

File: data/urdf/BioloidGP/BioloidGP.URDF (robot description, URDF)
Before this commit: robot BioloidGP, 17 links, 16 joints
Links:
- link torso: geometry collision mesh filename=torsoNoBattery.obj; visual mesh filename=torsoNoBattery.obj
